File: pcb/ledstipdimmer_panel.kicad_pcb (KiCad board)
At the start: 2 copper layers, 100 x 96 mm, 492 parts, among them P1 SolderCable, P2 SolderCable, Q1 NTTFS5820NLTAG, Q2 NTTFS5820NLTAG, U1 TPS7B6950, U2 IQS904D

Commit message: Production adjustments for Aetzwerk (Solder Resist with reduces for enhanced quality).
Other:
- rule pad_to_mask_clearance: 0.1 -> 0.05
- rule solder_mask_min_width: 0.2 -> 0.1
Changed lines of the file:
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@@
-(kicad_pcb (version 4) (host pcbnew 4.0.2+dfsg1-stable)
+(kicad_pcb (version 4) (host pcbnew 4.0.4-stable)
   (general
     (links 1164)
     (no_connects 144)
-    (area 64.117856 19.599999 176.382144 116.400001)
+    (area 64.192856 19.599999 176.307144 116.400001)
     (thickness 1.6)
     (drawings 133)
@@
     (pad_size 1.6 1.6)
     (pad_drill 0)
-    (pad_to_mask_clearance 0.1)
-    (solder_mask_min_width 0.2)
+    (pad_to_mask_clearance 0.05)
+    (solder_mask_min_width 0.1)
+    (pad_to_paste_clearance -0.03)
     (aux_axis_origin 0 0)
-    (visible_elements FFFFFF7F)
+    (visible_elements 7FFFFFFF)
     (pcbplotparams
       (layerselection 0x010f8_80000001)
